File: STM32_DEVBOARD_PCB/STM32_DEVBOARD/STM32_DEVBOARD.kicad_sch (KiCad schematic)
At the start: 60 parts, among them J1 GT-USB-7002C, J1 Screw_Terminal_01x02, J2 SWD, J4 Conn_01x03_Pin, Q1 AO3401A, SW1 BTN_RSET, SW2 BTN1, U1 STM32F401RCTx, U2 USBLC6-2P6, U3 LIS2DW12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

Commit message: Update symbols and check USB
Connections:
- net +3.3V: now also C19.1, C20.1, C21.1, D3.2 (A), J4.3 (Pin_3), R13.1, R14.1, R3.1, U3.10 (Vdd_IO), U3.2 (~{CS}), U3.9 (Vdd)
- net +3V3: no longer C19.1, C20.1, C21.1, D3.2 (A), J4.3 (Pin_3), R13.1, R14.1, R3.1, U3.10 (Vdd_IO), U3.2 (~{CS}), U3.9 (Vdd)
- no-connect marks 14 -> 51
Other:
- note added: "Limit crystal drive level"
- note added: "Vmeas = (32k * Vin) / 252k Vmeas = 3.0476v @Vin = 24v"
- moved on the sheet: C10, C12, C2, C3, C5, C6, C7, C8, C9, L2, R1, Y1
