File: STM32_DEVBOARD_PCB/STM32_DEVBOARD/STM32_DEVBOARD.kicad_sch (KiCad schematic)
At the start: 60 parts, among them J1 Screw_Terminal_01x02, J2 SWD, J2 USB_C_Receptacle_USB2.0, J4 Conn_01x03_Pin, Q1 AO3401A, SW1 BTN_RSET, SW2 BTN1, U1 USBLC6-2P6, U2 TPMP2359DJ, U3 STM32F401RCTx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

Commit message: Added images of render
Parts:
- added H1, H2: MountingHole, MountingHole:MountingHole_4.3mm_M4_Pad, symbol Mechanical:MountingHole
- J2: footprint (none) -> Connector_USB:USB_C_Receptacle_HRO_TYPE-C-31-M-12; JLC (none) -> C165948
Changed lines of the file:
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@@
     (stroke (width 0) (type default))
   )
-  (rectangle (start 175.26 15.24) (end 266.7 66.675)
+  (rectangle (start 173.99 15.24) (end 265.43 66.04)
     (stroke (width 0) (type default))
     (fill (type none))
   )
-  (rectangle (start 175.26 124.46) (end 266.7 280.67)
+  (rectangle (start 175.26 124.46) (end 265.43 280.67)
     (stroke (width 0) (type default))
     (fill (type none))
   )
-  (rectangle (start 267.97 121.92) (end 405.13 151.13)
+  (rectangle (start 267.97 123.19) (end 405.13 151.13)
     (stroke (width 0) (type default))
     (fill (type none))
@@
     (fill (type none))
   )
-  (rectangle (start 16.51 15.24) (end 173.99 123.19)
+  (rectangle (start 16.51 15.24) (end 172.72 121.92)
     (stroke (width 0) (type default))
     (fill (type none))
   )
-  (rectangle (start 175.26 96.52) (end 266.7 123.19)
+  (rectangle (start 175.26 96.52) (end 265.43 121.92)
     (stroke (width 0) (type default))
     (fill (type none))
   )
-  (rectangle (start 175.26 68.58) (end 266.7 95.25)
+  (rectangle (start 175.26 68.58) (end 265.43 93.98)
     (stroke (width 0) (type default))
     (fill (type none))
@@
     (fill (type none))
   )
-  (rectangle (start 16.51 242.57) (end 173.99 280.67)
+  (rectangle (start 16.51 242.57) (end 172.72 280.67)
     (stroke (width 0) (type default))
     (fill (type none))
   )
-  (rectangle (start 267.97 15.24) (end 405.13 73.66)
+  (rectangle (start 267.97 15.24) (end 405.13 72.39)
     (stroke (width 0) (type default))
     (fill (type none))
   )
-  (rectangle (start 16.51 124.46) (end 173.99 240.03)
+  (rectangle (start 16.51 124.46) (end 172.72 240.03)
     (stroke (width 0) (type default))
     (fill (type none))
   )
-  (rectangle (start 267.97 152.4) (end 405.13 180.34)
+  (rectangle (start 267.97 152.4) (end 405.13 179.07)
     (stroke (width 0) (type default))
     (fill (type none))
@@
     (effects (font (size 1 1)) (justify left bottom))
   )
-  (text "Connectors" (at 130.81 251.46 0)
+  (text "Connectors" (at 129.54 250.19 0)
     (effects (font (size 5 5) (thickness 0.6) bold) (justify left bottom))
   )
@@
       (effects (font (size 1.27 1.27)))
     )
-    (property "Footprint" "" (at 50.8 166.37 0)
-      (effects (font (size 1.27 1.27)) hide)
-    )
-    (property "Datasheet" "https://www.usb.org/sites/default/files/documents/usb_type-c.zip" (at 50.8 166.37 0)
+    (property "Footprint" "Connector_USB:USB_C_Receptacle_HRO_TYPE-C-31-M-12" (at 50.8 166.37 0)
+      (effects (font (size 1.27 1.27)) hide)
+    )
+    (property "Datasheet" "C165948" (at 50.8 166.37 0)
+      (effects (font (size 1.27 1.27)) hide)
+    )
+    (property "JLC" "C165948" (at 46.99 166.37 0)
       (effects (font (size 1.27 1.27)) hide)
     )
@@
         (path "/c729864e-51f7-4d56-a7a2-194af487a099"
           (reference "SW1") (unit 1)
+        )
+      )
+    )
+  )
+  (symbol (lib_id "Mechanical:MountingHole") (at 114.3 261.62 0) (unit 1)
+    (in_bom yes) (on_board yes) (dnp no) (fields_autoplaced)
+    (property "Reference" "H2" (at 116.84 260.985 0)
+      (effects (font (size 1.27 1.27)) (justify left))
+    )
+    (property "Value" "MountingHole" (at 116.84 263.525 0)
+      (effects (font (size 1.27 1.27)) (justify left))
+    )
+    (property "Footprint" "MountingHole:MountingHole_4.3mm_M4_Pad" (at 114.3 261.62 0)
+      (effects (font (size 1.27 1.27)) hide)
+    )
+    (property "Datasheet" "~" (at 114.3 261.62 0)
+      (effects (font (size 1.27 1.27)) hide)
+    )
+    (instances
+      (project "STM32_DEVBOARD"
+        (path "/c729864e-51f7-4d56-a7a2-194af487a099"
+          (reference "H2") (unit 1)
         )
       )
@@
         )
       )
+    )
+  )
+  (symbol (lib_id "Mechanical:MountingHole") (at 114.3 255.27 0) (unit 1)
+    (in_bom yes) (on_board yes) (dnp no)
+    (property "Reference" "H1" (at 116.84 254.635 0)
+      (effects (font (size 1.27 1.27)) (justify left))
+    )
+    (property "Value" "MountingHole" (at 116.84 257.175 0)
+      (effects (font (size 1.27 1.27)) (justify left))
+    )
+    (property "Footprint" "MountingHole:MountingHole_4.3mm_M4_Pad" (at 114.3 255.27 0)
+      (effects (font (size 1.27 1.27)) hide)
+    )
+    (property "Datasheet" "~" (at 114.3 255.27 0)
+      (effects (font (size 1.27 1.27)) hide)
+    )
+    (instances
+      (project "STM32_DEVBOARD"
+        (path "/c729864e-51f7-4d56-a7a2-194af487a099"
+          (reference "H1") (unit 1)
+        )
+      )

Commit message: Updates to board and start to populate BOM
Parts:
- C10: LCSC Part # (none) -> C19666
- FB1: JLC C1017 -> (none); LCSC Part # (none) -> C1017
- J2: JLC C165948 -> (none); LCSC Part # (none) -> C165948
- R12, R14: LCSC Part # (none) -> C319937
- R4: LCSC Part # C22809 -> C319937
- R6, R7: LCSC Part # (none) -> C2692696
- R9: LCSC Part # C22843 -> C319937
- U1: LCSC Part # (none) -> C15999
- U3: LCSC Part # (none) -> C74524
- U4: LCSC Part # (none) -> C92489
- U5: LCSC Part # (none) -> C189624
- Y1: JLCPCB C13738 -> (none); LCSC Part # (none) -> C13738
Changed lines of the file:
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@@
       (effects (font (size 1.27 1.27)) hide)
     )
-    (property "Datasheet" "C165948" (at 50.8 166.37 0)
+    (property "Datasheet" "" (at 50.8 166.37 0)
       (effects (font (size 1.27 1.27)) hide)
     )
-    (property "JLC" "C165948" (at 46.99 166.37 0)
+    (property "JLC" "" (at 46.99 166.37 0)
+      (effects (font (size 1.27 1.27)) hide)
+    )
+    (property "LCSC Part #" "C165948" (at 46.99 166.37 0)
       (effects (font (size 1.27 1.27)) hide)
     )
@@
       (effects (font (size 1.27 1.27)) hide)
     )
+    (property "LCSC Part #" "C92489" (at 302.26 97.79 0)
+      (effects (font (size 1.27 1.27)) hide)
+    )
     (pin "1")
     (pin "2")
@@
       (effects (font (size 1.27 1.27)) hide)
     )
+    (property "LCSC Part #" "C319937" (at 290.83 31.75 0)
+      (effects (font (size 1.27 1.27)) hide)
+    )
     (pin "1")
     (pin "2")
@@
       (effects (font (size 1.27 1.27)) hide)
     )
+    (property "LCSC Part #" "C19666" (at 196.85 256.54 0)
+      (effects (font (size 1.27 1.27)) hide)
+    )
     (pin "1")
     (pin "2")
@@
       (effects (font (size 1.27 1.27)) hide)
     )
-    (property "JLCPCB" "C13738" (at 189.23 39.37 0)
+    (property "JLCPCB" "" (at 189.23 39.37 0)
+      (effects (font (size 1.27 1.27)) hide)
+    )
+    (property "LCSC Part #" "C13738" (at 189.23 39.37 0)
       (effects (font (size 1.27 1.27)) hide)
     )
@@
       (effects (font (size 1.27 1.27)) hide)
     )
+    (property "LCSC Part #" "C15999" (at 107.95 214.63 0)
+      (effects (font (size 1.27 1.27)) hide)
+    )
     (pin "1")
     (pin "2")
@@
       (effects (font (size 1.27 1.27)) hide)
     )
+    (property "LCSC Part #" "C2692696" (at 107.95 181.61 0)
+      (effects (font (size 1.27 1.27)) hide)
+    )
     (pin "1")
     (pin "2")
@@
       (effects (font (size 1.27 1.27)) hide)
     )
-    (property "JLC" "C1017" (at 72.39 40.64 90)
+    (property "JLC" "" (at 72.39 40.64 90)
+      (effects (font (size 1.27 1.27)) hide)
+    )
+    (property "LCSC Part #" "C1017" (at 72.39 40.64 0)
       (effects (font (size 1.27 1.27)) hide)
     )
@@
       (effects (font (size 1.27 1.27)) hide)
     )
+    (property "LCSC Part #" "C189624" (at 308.61 44.45 0)
+      (effects (font (size 1.27 1.27)) hide)
+    )
     (pin "1")
     (pin "10")
@@
       (effects (font (size 1.27 1.27)) hide)
     )
+    (property "LCSC Part #" "C74524" (at 217.17 222.25 0)
+      (effects (font (size 1.27 1.27)) hide)
+    )
     (pin "1")
     (pin "10")
@@
       (effects (font (size 1.27 1.27)) hide)
     )
-    (property "LCSC Part #" "C22809" (at 118.11 83.82 0)
+    (property "LCSC Part #" "C319937" (at 118.11 83.82 0)
       (effects (font (size 1.27 1.27)) hide)
     )
@@
       (effects (font (size 1.27 1.27)) hide)
     )
-    (property "LCSC Part #" "C22843" (at 290.83 205.74 0)
+    (property "LCSC Part #" "C319937" (at 290.83 205.74 0)
       (effects (font (size 1.27 1.27)) hide)
     )
@@
       (effects (font (size 1.27 1.27)) hide)
     )
+    (property "LCSC Part #" "C319937" (at 288.29 31.75 0)
+      (effects (font (size 1.27 1.27)) hide)
+    )
     (pin "1")
     (pin "2")
@@
       (effects (font (size 1.27 1.27)) hide)
     )
+    (property "LCSC Part #" "C2692696" (at 107.95 163.83 0)
+      (effects (font (size 1.27 1.27)) hide)
+    )

Commit message: Added PCB render
Parts:
- added TP1: GND, TestPoint:TestPoint_Pad_D2.0mm, symbol Connector:TestPoint
- added TP2: 3.3V, TestPoint:TestPoint_Pad_D2.0mm, symbol Connector:TestPoint
- added TP3: 5V, TestPoint:TestPoint_Pad_D2.0mm, symbol Connector:TestPoint
- added TP4: 24V, TestPoint:TestPoint_Pad_D2.0mm, symbol Connector:TestPoint
Connections:
- net +24V: now also TP4.1
- net +3.3V: now also TP2.1
- net +5V: now also TP3.1
- net GND: now also TP1.1
Changed lines of the file:
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@@
     (stroke (width 0) (type default))
   )
+  (wire (pts (xy 290.83 233.68) (xy 290.83 234.95))
+    (stroke (width 0) (type default))
+  )
   (wire (pts (xy 41.91 55.88) (xy 41.91 57.15))
     (stroke (width 0) (type default))
@@
     (stroke (width 0) (type default))
   )
+  (wire (pts (xy 302.26 232.41) (xy 302.26 233.68))
+    (stroke (width 0) (type default))
+  )
   (wire (pts (xy 299.72 82.55) (xy 304.8 82.55))
     (stroke (width 0) (type default))
@@
     (stroke (width 0) (type default))
   )
+  (wire (pts (xy 314.96 232.41) (xy 314.96 233.68))
+    (stroke (width 0) (type default))
+  )
   (wire (pts (xy 181.61 76.2) (xy 181.61 77.47))
     (stroke (width 0) (type default))
@@
     (stroke (width 0) (type default))
   )
+  (wire (pts (xy 326.39 232.41) (xy 326.39 233.68))
+    (stroke (width 0) (type default))
+  )
   (wire (pts (xy 209.55 77.47) (xy 209.55 78.74))
     (stroke (width 0) (type default))
@@
     )
   )
+  (symbol (lib_id "power:+24V") (at 326.39 232.41 0) (unit 1)
+    (in_bom yes) (on_board yes) (dnp no) (fields_autoplaced)
+    (property "Reference" "#PWR048" (at 326.39 236.22 0)
+      (effects (font (size 1.27 1.27)) hide)
+    )
+    (property "Value" "+24V" (at 326.39 228.6 0)
+      (effects (font (size 1.27 1.27)))
+    )
+    (property "Footprint" "" (at 326.39 232.41 0)
+      (effects (font (size 1.27 1.27)) hide)
+    )
+    (property "Datasheet" "" (at 326.39 232.41 0)
+      (effects (font (size 1.27 1.27)) hide)
+    )
+    (pin "1")
+    (instances
+      (project "STM32_DEVBOARD"
+        (path "/c729864e-51f7-4d56-a7a2-194af487a099"
+          (reference "#PWR048") (unit 1)
+        )
+      )
+    )
+  )
   (symbol (lib_id "Device:C_Small") (at 120.65 102.87 270) (unit 1)
     (in_bom yes) (on_board yes) (dnp no)
@@
     )
   )
+  (symbol (lib_id "Connector:TestPoint") (at 302.26 233.68 180) (unit 1)
+    (in_bom yes) (on_board yes) (dnp no)
+    (property "Reference" "TP2" (at 307.34 237.49 0)
+      (effects (font (size 1.27 1.27)) (justify left))
+    )
+    (property "Value" "3.3V" (at 307.34 240.03 0)
+      (effects (font (size 1.27 1.27)) (justify left))
+    )
+    (property "Footprint" "TestPoint:TestPoint_Pad_D2.0mm" (at 297.18 233.68 0)
+      (effects (font (size 1.27 1.27)) hide)
+    )
+    (property "Datasheet" "~" (at 297.18 233.68 0)
+      (effects (font (size 1.27 1.27)) hide)
+    )
+    (pin "1")
+    (instances
+      (project "STM32_DEVBOARD"
+        (path "/c729864e-51f7-4d56-a7a2-194af487a099"
+          (reference "TP2") (unit 1)
+        )
+      )
+    )
+  )
   (symbol (lib_id "power:PWR_FLAG") (at 71.12 96.52 0) (unit 1)
     (in_bom yes) (on_board yes) (dnp no) (fields_autoplaced)
@@
     )
   )
+  (symbol (lib_id "power:+3.3V") (at 302.26 232.41 0) (unit 1)
+    (in_bom yes) (on_board yes) (dnp no) (fields_autoplaced)
+    (property "Reference" "#PWR047" (at 302.26 236.22 0)
+      (effects (font (size 1.27 1.27)) hide)
+    )
+    (property "Value" "+3.3V" (at 302.26 228.6 0)
+      (effects (font (size 1.27 1.27)))
+    )
+    (property "Footprint" "" (at 302.26 232.41 0)
+      (effects (font (size 1.27 1.27)) hide)
+    )
+    (property "Datasheet" "" (at 302.26 232.41 0)
+      (effects (font (size 1.27 1.27)) hide)
+    )
+    (pin "1")
+    (instances
+      (project "STM32_DEVBOARD"
+        (path "/c729864e-51f7-4d56-a7a2-194af487a099"
+          (reference "#PWR047") (unit 1)
+        )
+      )
+    )
+  )
   (symbol (lib_id "power:PWR_FLAG") (at 27.94 252.73 0) (unit 1)
     (in_bom yes) (on_board yes) (dnp no) (fields_autoplaced)
@@
     )
   )
+  (symbol (lib_id "power:GND") (at 290.83 234.95 0) (unit 1)
+    (in_bom yes) (on_board yes) (dnp no) (fields_autoplaced)
+    (property "Reference" "#PWR049" (at 290.83 241.3 0)
+      (effects (font (size 1.27 1.27)) hide)
+    )
+    (property "Value" "GND" (at 290.83 240.03 0)
+      (effects (font (size 1.27 1.27)))
+    )
+    (property "Footprint" "" (at 290.83 234.95 0)
+      (effects (font (size 1.27 1.27)) hide)
+    )
+    (property "Datasheet" "" (at 290.83 234.95 0)
+      (effects (font (size 1.27 1.27)) hide)
+    )
+    (pin "1")
+    (instances
+      (project "STM32_DEVBOARD"
+        (path "/c729864e-51f7-4d56-a7a2-194af487a099"
+          (reference "#PWR049") (unit 1)
+        )
+      )
+    )
+  )
   (symbol (lib_id "power:+3.3V") (at 118.11 72.39 0) (unit 1)
     (in_bom yes) (on_board yes) (dnp no) (fields_autoplaced)
@@
     )
   )
+  (symbol (lib_id "Connector:TestPoint") (at 290.83 233.68 0) (unit 1)
+    (in_bom yes) (on_board yes) (dnp no)
+    (property "Reference" "TP1" (at 285.75 229.87 0)
+      (effects (font (size 1.27 1.27)) (justify left))
+    )
+    (property "Value" "GND" (at 285.75 232.41 0)
+      (effects (font (size 1.27 1.27)) (justify left))
+    )
+    (property "Footprint" "TestPoint:TestPoint_Pad_D2.0mm" (at 295.91 233.68 0)
+      (effects (font (size 1.27 1.27)) hide)
+    )
+    (property "Datasheet" "~" (at 295.91 233.68 0)
+      (effects (font (size 1.27 1.27)) hide)
+    )
+    (pin "1")
+    (instances
+      (project "STM32_DEVBOARD"
+        (path "/c729864e-51f7-4d56-a7a2-194af487a099"
+          (reference "TP1") (unit 1)
+        )
+      )
+    )
+  )
   (symbol (lib_id "Device:C_Small") (at 99.06 38.1 0) (unit 1)
     (in_bom yes) (on_board yes) (dnp no)
@@
     )
   )
+  (symbol (lib_id "Connector:TestPoint") (at 314.96 233.68 180) (unit 1)
+    (in_bom yes) (on_board yes) (dnp no)
+    (property "Reference" "TP3" (at 320.04 237.49 0)
+      (effects (font (size 1.27 1.27)) (justify left))
+    )
+    (property "Value" "5V" (at 318.77 240.03 0)
+      (effects (font (size 1.27 1.27)) (justify left))
+    )
+    (property "Footprint" "TestPoint:TestPoint_Pad_D2.0mm" (at 309.88 233.68 0)
+      (effects (font (size 1.27 1.27)) hide)
+    )
+    (property "Datasheet" "~" (at 309.88 233.68 0)
+      (effects (font (size 1.27 1.27)) hide)
+    )
+    (pin "1")
+    (instances
+      (project "STM32_DEVBOARD"
+        (path "/c729864e-51f7-4d56-a7a2-194af487a099"
+          (reference "TP3") (unit 1)
+        )
+      )
+    )
+  )
   (symbol (lib_id "Switch:SW_Push") (at 278.13 165.1 90) (unit 1)
     (in_bom yes) (on_board yes) (dnp no) (fields_autoplaced)
@@
     )
   )
+  (symbol (lib_id "Connector:TestPoint") (at 326.39 233.68 180) (unit 1)
+    (in_bom yes) (on_board yes) (dnp no)
+    (property "Reference" "TP4" (at 331.47 237.49 0)
+      (effects (font (size 1.27 1.27)) (justify left))
+    )
+    (property "Value" "24V" (at 330.2 240.03 0)
+      (effects (font (size 1.27 1.27)) (justify left))
+    )
+    (property "Footprint" "TestPoint:TestPoint_Pad_D2.0mm" (at 321.31 233.68 0)
+      (effects (font (size 1.27 1.27)) hide)
+    )
+    (property "Datasheet" "~" (at 321.31 233.68 0)
+      (effects (font (size 1.27 1.27)) hide)
+    )
+    (pin "1")
+    (instances
+      (project "STM32_DEVBOARD"
+        (path "/c729864e-51f7-4d56-a7a2-194af487a099"
+          (reference "TP4") (unit 1)
+        )
+      )
+    )
+  )
   (symbol (lib_id "Device:C_Small") (at 281.94 85.09 0) (unit 1)
     (in_bom yes) (on_board yes) (dnp no) (fields_autoplaced)
@@
         )
       )
+    )
+  )
+  (symbol (lib_id "power:+5V") (at 314.96 232.41 0) (unit 1)
+    (in_bom yes) (on_board yes) (dnp no) (fields_autoplaced)
+    (property "Reference" "#PWR050" (at 314.96 236.22 0)
+      (effects (font (size 1.27 1.27)) hide)
+    )
+    (property "Value" "+5V" (at 314.96 228.6 0)
+      (effects (font (size 1.27 1.27)))
+    )
+    (property "Footprint" "" (at 314.96 232.41 0)
+      (effects (font (size 1.27 1.27)) hide)
+    )
+    (property "Datasheet" "" (at 314.96 232.41 0)
+      (effects (font (size 1.27 1.27)) hide)
+    )
+    (pin "1")
+    (instances
+      (project "STM32_DEVBOARD"
+        (path "/c729864e-51f7-4d56-a7a2-194af487a099"
+          (reference "#PWR050") (unit 1)
+        )
+      )

Commit message: Remove files
Other:
- note added: "Test Points"
Changed lines of the file:
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@@
+    (fill (type none))
+  )
+  (rectangle (start 267.97 222.25) (end 405.13 250.19)
+    (stroke (width 0) (type default))
     (fill (type none))
   )
@@
     (effects (font (size 5 5) (thickness 0.6) bold) (justify left bottom))
   )
+  (text "Test Points" (at 360.68 229.87 0)
+    (effects (font (size 5 5) (thickness 0.6) bold) (justify left bottom))
+  )
