File: STM32_DEVBOARD_PCB/STM32_DEVBOARD/STM32_DEVBOARD.kicad_sch (KiCad schematic)
At the start: 69 parts, among them J1 Screw_Terminal_01x02, J2 SWD, J2 USB_C_Receptacle_USB2.0, J4 Conn_01x03_Pin, Q1 AO3401A, Q3 MMBT3904, SW1 BTN_RSET, SW2 BTN1, U1 USBLC6-2P6, U2 TPMP2359DJ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

Commit message: updated firmware examples
Parts:
- BZ1: LCSC Part # C201040 -> C96256
- J4: LCSC Part # C5142365 -> C49257
Changed lines of the file:
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@@
     (stroke (width 0) (type default))
   )
-  (rectangle (start 173.99 15.24) (end 265.43 66.04)
+  (rectangle (start 175.26 15.24) (end 265.43 66.04)
     (stroke (width 0) (type default))
     (fill (type none))
@@
       (effects (font (size 1.27 1.27)) hide)
     )
+    (property "Sim.Device" "D" (at 50.8 45.72 0)
+      (effects (font (size 1.27 1.27)) hide)
+    )
+    (property "Sim.Pins" "1=A 2=K" (at 50.8 45.72 0)
+      (effects (font (size 1.27 1.27)) hide)
+    )
     (pin "1")
     (pin "2")
@@
       (effects (font (size 1.27 1.27)) hide)
     )
+    (property "Sim.Device" "R" (at 62.23 40.64 0)
+      (effects (font (size 1.27 1.27)) hide)
+    )
+    (property "Sim.Pins" "1=+ 2=-" (at 62.23 40.64 0)
+      (effects (font (size 1.27 1.27)) hide)
+    )
+    (property "Sim.Params" "r=0" (at 62.23 40.64 0)
+      (effects (font (size 1.27 1.27)) hide)
+    )
     (pin "1")
     (pin "2")
@@
       (effects (font (size 1.27 1.27)) hide)
     )
-    (property "LCSC Part #" "C5142365" (at 201.93 138.43 0)
+    (property "LCSC Part #" "C49257" (at 201.93 138.43 0)
       (effects (font (size 1.27 1.27)) hide)
     )
@@
       (effects (font (size 1.27 1.27)) hide)
     )
+    (property "Sim.Device" "R" (at 41.91 53.34 0)
+      (effects (font (size 1.27 1.27)) hide)
+    )
+    (property "Sim.Pins" "1=+ 2=-" (at 41.91 53.34 0)
+      (effects (font (size 1.27 1.27)) hide)
+    )
     (pin "1")
     (pin "2")
@@
       (effects (font (size 1.27 1.27)) hide)
     )
-    (property "LCSC Part #" "C201040" (at 303.53 227.33 0)
+    (property "LCSC Part #" "C96256" (at 303.53 227.33 0)
       (effects (font (size 1.27 1.27)) hide)
     )
@@
       (effects (font (size 1.27 1.27)) hide)
     )
+    (property "Sim.Device" "PMOS" (at 41.91 43.18 0)
+      (effects (font (size 1.27 1.27)) hide)
+    )
+    (property "Sim.Type" "VDMOS" (at 41.91 43.18 0)
+      (effects (font (size 1.27 1.27)) hide)
+    )
+    (property "Sim.Pins" "1=D 2=G 3=S" (at 41.91 43.18 0)
+      (effects (font (size 1.27 1.27)) hide)
+    )
