File: STM32_DEVBOARD_PCB/STM32_DEVBOARD/_autosave-STM32_DEVBOARD.kicad_sch (KiCad schematic)
At the start: 60 parts, among them J1 Screw_Terminal_01x02, J2 SWD, J2 USB_C_Receptacle_USB2.0, J4 Conn_01x03_Pin, Q1 AO3401A, SW1 BTN_RSET, SW2 BTN1, U1 USBLC6-2P6, U2 TPMP2359DJ, U3 STM32F401RCTx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

Commit message: Added USB C connector and tidy up traces.
Parts:
- J2: footprint (none) -> Connector_USB:USB_C_Receptacle_HRO_TYPE-C-31-M-12; JLC (none) -> C165948
Changed lines of the file:
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@@
       (effects (font (size 1.27 1.27)))
     )
-    (property "Footprint" "" (at 50.8 166.37 0)
+    (property "Footprint" "Connector_USB:USB_C_Receptacle_HRO_TYPE-C-31-M-12" (at 50.8 166.37 0)
       (effects (font (size 1.27 1.27)) hide)
     )
-    (property "Datasheet" "https://www.usb.org/sites/default/files/documents/usb_type-c.zip" (at 50.8 166.37 0)
+    (property "Datasheet" "C165948" (at 50.8 166.37 0)
       (effects (font (size 1.27 1.27)) hide)
     )
+    (property "JLC" "C165948" (at 46.99 166.37 0)
+      (effects (font (size 1.27 1.27)) hide)
+    )
