File: STM32_DEVBOARD_PCB/STM32_DEVBOARD/_autosave-STM32_DEVBOARD.kicad_sch (KiCad schematic)
At the start: 69 parts, among them J1 Screw_Terminal_01x02, J2 SWD, J2 USB_C_Receptacle_USB2.0, J4 Conn_01x03_Pin, Q1 AO3401A, Q3 MMBT3904, SW1 BTN_RSET, SW2 BTN1, U1 USBLC6-2P6, U2 TPMP2359DJ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

Commit message: V1
Parts:
- BZ1: LCSC Part # C201040 -> C96256
- J4: LCSC Part # C5142365 -> C49257
Changed lines of the file:
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@@
       (effects (font (size 1.27 1.27)) hide)
     )
-    (property "LCSC Part #" "C5142365" (at 201.93 138.43 0)
+    (property "LCSC Part #" "C49257" (at 201.93 138.43 0)
       (effects (font (size 1.27 1.27)) hide)
     )
@@
       (effects (font (size 1.27 1.27)) hide)
     )
-    (property "LCSC Part #" "C201040" (at 303.53 227.33 0)
-      (effects (font (size 1.27 1.27)) hide)
-    )
+    (property "LCSC Part #" "C96256" (at 303.53 227.33 0)
+      (effects (font (size 1.27 1.27)) hide)
+    )
