File: STM32_DEVBOARD_PCB/STM32_DEVBOARD/STM32_DEVBOARD.kicad_pcb (KiCad board)
At the start: 2 copper layers, 60 x 106 mm, 62 parts, among them J1 Screw_Terminal_01x02, J2 USB_C_Receptacle_USB2.0, J3 SWD, J4 Conn_01x03_Pin, Q1 AO3401A, SW1 BTN_RSET, SW2 BTN1, U1 USBLC6-2P6, U2 TPMP2359DJ, U3 STM32F401RCTx, U4 BME280, U5 LIS2DW12, Y1 16MHz

Commit message: Remove files
Parts:
- added TP1: GND, TestPoint:TestPoint_Pad_D2.0mm, F.Cu at (63.2, 92.7)
- added TP2: 3.3V, TestPoint:TestPoint_Pad_D2.0mm, F.Cu at (63.2, 96.3)
- added TP3: 5V, TestPoint:TestPoint_Pad_D2.0mm, F.Cu at (63.2, 99.8)
- added TP4: 24V, TestPoint:TestPoint_Pad_D2.0mm, F.Cu at (71.9, 98.6)
Routing:
- net +24V: track 4.66 -> 9.06 mm
- net +5V: track 50.9 -> 54.8 mm
- net GND: track 96.9 -> 99.3 mm, vias 27 -> 28
Other:
- board text added: "24V"
- board text added: "5V"
