File: STM32_DEVBOARD_PCB/STM32_DEVBOARD/STM32_DEVBOARD.kicad_pcb (KiCad board)
At the start: 2 copper layers, 60 x 106 mm, 66 parts, among them J1 Screw_Terminal_01x02, J2 USB_C_Receptacle_USB2.0, J3 SWD, J4 Conn_01x03_Pin, Q1 AO3401A, SW1 BTN_RSET, SW2 BTN1, U1 USBLC6-2P6, U2 TPMP2359DJ, U3 STM32F401RCTx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

Commit message: V1
Parts:
- added BZ1: Buzzer, Buzzer_Beeper:MagneticBuzzer_CUI_CST-931RP-A, F.Cu at (63.5, 73.7)
- added Q3: MMBT3904, Package_TO_SOT_SMD:SOT-23, F.Cu at (75.9, 76.2)
- added R18: 1k, Resistor_SMD:R_0603_1608Metric, F.Cu at (78.7, 78.7)
- L1: footprint Inductor_SMD:L_0402_1005Metric -> Inductor_SMD:L_0603_1608Metric
- R10: footprint Resistor_SMD:R_0402_1005Metric -> Resistor_SMD:R_0603_1608Metric
- SW1, SW2: footprint Button_Switch_SMD:SW_Tactile_SPST_NO_Straight_CK_PTS636Sx25SMTRLFS -> STM32DEVBOARD:SW_Tactile_SPST_NO_Straight_CK_PTS636-SK25J-SMTR-LFS
- moved D4 45.0 mm to (80.8, 117.3), turned to 90 degrees
- moved R13 24.0 mm to (86.1, 94.5), turned to -90 degrees
- moved D2 0.51 mm to (78.7, 93.0)
- moved R10 0.51 mm to (89.8, 93.0)
- moved R1 0.43 mm to (74.7, 92.7)
- moved L1 0.25 mm to (74.7, 89.6)
Connections:
- U3 pad 16: unconnected-(U3-PA2-Pad16) -> BTN1
- U3 pad 2: LED -> unconnected-(U3-PC13-Pad2)
- U3 pad 36: unconnected-(U3-PB15-Pad36) -> BUZZ
- U3 pad 37: unconnected-(U3-PC6-Pad37) -> LED
Routing:
- net LED: track 4.00 -> 33.1 mm, vias 0 -> 2
- net Net-(D4-K): track 1.56 -> 25.6 mm, vias 0 -> 2
- net BUZZ: track 0.00 -> 18.9 mm, vias 0 -> 4
- net BTN1: track 4.48 -> 22.7 mm
- net Net-(BZ1-+): track 0.00 -> 14.2 mm
- net +3.3V: track 86.1 -> 81.4 mm
- net GND: track 99.3 -> 103.1 mm
- net Net-(Q3-B): track 0.00 -> 2.15 mm
- net SPI1_MISO: track 7.11 -> 5.84 mm
- net +5V: track 54.8 -> 53.6 mm
- net Net-(D2-A): track 11.0 -> 11.9 mm
Other:
- board text added: "JLCJLCJLCJLC"
